File: llm-kicad/02_usb_hub_control.kicad_sch (KiCad schematic)
At the start: 22 parts, among them J1 TYPE-C-31-M-12, Q6 BSS138P,215, Q7 BSS138P,215, U1 CH334F, U2 CP2102N-A02-GQFN28, U9 TPD4E05U06DQA, Y1 12MHz X322512MSB4SI

Commit message: More progress
Parts:
- removed Y1: 12MHz X322512MSB4SI, Crystal:Crystal_SMD_3225-4Pin_3.2x2.5mm, symbol Device:Crystal
- added C28: 100nF, Capacitor_SMD:C_0402_1005Metric, symbol Device:C
- added Y1: Crystal 12MHz, Crystal:Crystal_SMD_3225-4Pin_3.2x2.5mm, symbol Device:Crystal_GND24
- C23, C25: value 1uF 25V -> 4.7uF 25V; footprint Capacitor_SMD:C_0402_1005Metric -> Capacitor_SMD:C_0805_2012Metric; LCSC C52923 -> C1779
- R35: LCSC C11702 -> C25744
- U1: footprint Package_DFN_QFN:QFN-24-1EP_3x4mm_P0.4mm_EP1.65x2.65mm_ThermalVias -> Package_DFN_QFN:QFN-24-1EP_4x4mm_P0.5mm_EP2.6x2.6mm_ThermalVias
Connections:
- net +3.3V: now also C28.1
- net GND: now also C28.2, Y1.2 (G), Y1.4 (G)
- net HIL_CC_EN_N: now also U2.17 (RS485/GPIO.2); no longer U2.20 (GPIO.6)
- net HIL_DATA_EN_N: now also U2.22 (GPIO.4); no longer U2.21 (GPIO.5)
- net HIL_VBUS_EN: now also U2.20 (GPIO.6); no longer U2.22 (GPIO.4)
- net J1_CC1: now also U9.7 (NC)
- net J1_CC2: now also U9.6 (NC)
- net J1_D+: now also U9.9 (NC)
- net J1_D-: now also U9.10 (NC)
- net VBUS_HIL_SNS: now also U2.18 (~{RXT}/GPIO.1); no longer U2.17 (RS485/GPIO.2)
- net VBUS_PWR_SNS: now also U2.16 (~{WAKEUP}/GPIO.3); no longer U2.18 (~{RXT}/GPIO.1)
- net VBUS_UP_SNS: now also U2.21 (GPIO.5); no longer U2.16 (~{WAKEUP}/GPIO.3)
- net at U1.3 (XO): now also Y1.3
- net at U1.4 (XI): now also Y1.1
- no-connect marks 31 -> 25
Other:
- note added: "Near VDD (pin8)"
- note added: "Near VREGIN (pin7)"
- moved on the sheet: C23, C24, C25
