File: llm-kicad/03_dut_interface.kicad_sch (KiCad schematic)
At the start: 10 parts, among them J3 TYPE-C-31-M-12, U10 TPD4E05U06DQA, U5 TS3USB221A, U6 SN74LVC1G125DBVR

Commit message: More progress
Connections:
- net J3_CC1: now also U10.7 (NC)
- net J3_CC2: now also U10.6 (NC)
- net J3_D+: now also U10.2 (D1-), U10.9 (NC), U5.8 (D+); no longer U10.1 (D1+), U5.1 (1D+)
- net J3_D-: now also U10.1 (D1+), U10.10 (NC), U5.7 (D-); no longer U10.2 (D1-), U5.2 (1D-)
- net U1_P2_D+: now also U5.1 (1D+); no longer U5.8 (D+)
- net U1_P2_D-: now also U5.2 (1D-); no longer U5.7 (D-)
- no-connect marks 8 -> 4
Changed lines of the file:
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@@
-	)
-	(no_connect
-		(at 40.64 88.9)
-	)
-	(no_connect
-		(at 40.64 104.14)
-	)
-	(no_connect
-		(at 66.04 88.9)
 	)
 	(no_connect
@@
 	)
 	(no_connect
-		(at 66.04 104.14)
-	)
-	(no_connect
 		(at 48.26 48.26)
 	)
@@
 	(wire
 		(pts
+			(xy 66.04 104.14) (xy 67.31 104.14)
+		)
+		(stroke
+			(width 0)
+			(type default)
+		)
+	)
+	(wire
+		(pts
 			(xy 46.99 55.88) (xy 46.99 53.34)
 		)
@@
 	(wire
 		(pts
+			(xy 73.66 43.18) (xy 76.2 43.18)
+		)
+		(stroke
+			(width 0)
+			(type default)
+		)
+	)
+	(wire
+		(pts
 			(xy 191.77 110.49) (xy 191.77 107.95)
 		)
@@
 	(wire
 		(pts
+			(xy 39.37 93.98) (xy 40.64 93.98)
+		)
+		(stroke
+			(width 0)
+			(type default)
+		)
+	)
+	(wire
+		(pts
 			(xy 234.95 71.12) (xy 234.95 67.31)
 		)
@@
 	(wire
 		(pts
+			(xy 39.37 99.06) (xy 40.64 99.06)
+		)
+		(stroke
+			(width 0)
+			(type default)
+		)
+	)
+	(wire
+		(pts
 			(xy 208.28 87.63) (xy 208.28 95.25)
 		)
@@
 	(wire
 		(pts
-			(xy 73.66 43.18) (xy 76.2 43.18)
+			(xy 46.99 43.18) (xy 48.26 43.18)
 		)
 		(stroke
@@
 	(wire
 		(pts
+			(xy 46.99 40.64) (xy 48.26 40.64)
+		)
+		(stroke
+			(width 0)
+			(type default)
+		)
+	)
+	(wire
+		(pts
 			(xy 208.28 76.2) (xy 208.28 80.01)
 		)
@@
 	(wire
 		(pts
+			(xy 39.37 104.14) (xy 40.64 104.14)
+		)
+		(stroke
+			(width 0)
+			(type default)
+		)
+	)
+	(wire
+		(pts
 			(xy 191.77 102.87) (xy 190.5 102.87)
 		)
@@
 	(wire
 		(pts
+			(xy 67.31 99.06) (xy 66.04 99.06)
+		)
+		(stroke
+			(width 0)
+			(type default)
+		)
+	)
+	(wire
+		(pts
 			(xy 111.76 48.26) (xy 111.76 50.8)
 		)
@@
 	(wire
 		(pts
+			(xy 67.31 93.98) (xy 66.04 93.98)
+		)
+		(stroke
+			(width 0)
+			(type default)
+		)
+	)
+	(wire
+		(pts
 			(xy 99.06 50.8) (xy 111.76 50.8)
 		)
@@
 	(wire
 		(pts
+			(xy 39.37 88.9) (xy 40.64 88.9)
+		)
+		(stroke
+			(width 0)
+			(type default)
+		)
+	)
+	(wire
+		(pts
 			(xy 167.64 129.54) (xy 167.64 130.81)
 		)
@@
 		(pts
 			(xy 240.03 71.12) (xy 240.03 67.31)
+		)
+		(stroke
+			(width 0)
+			(type default)
+		)
+	)
+	(wire
+		(pts
+			(xy 66.04 88.9) (xy 67.31 88.9)
 		)
 		(stroke
@@
 	)
 	(label "J3_D+"
-		(at 48.26 40.64 180)
-		(effects
-			(font
-				(size 1.27 1.27)
-			)
-			(justify right bottom)
+		(at 76.2 43.18 0)
+		(effects
+			(font
+				(size 1.27 1.27)
+			)
+			(justify left bottom)
+		)
+	)
+	(label "J3_CC1"
+		(at 67.31 88.9 0)
+		(effects
+			(font
+				(size 1.27 1.27)
+			)
+			(justify left bottom)
 		)
 	)
@@
 	)
 	(label "J3_CC2"
-		(at 66.04 99.06 0)
+		(at 67.31 99.06 0)
+		(effects
+			(font
+				(size 1.27 1.27)
+			)
+			(justify left bottom)
+		)
+	)
+	(label "J3_CC2"
+		(at 67.31 104.14 0)
 		(effects
 			(font
@@
 	)
 	(label "J3_D-"
-		(at 40.64 99.06 180)
+		(at 39.37 88.9 180)
 		(effects
 			(font
@@
 		)
 	)
+	(label "J3_D-"
+		(at 39.37 93.98 180)
+		(effects
+			(font
+				(size 1.27 1.27)
+			)
+			(justify right bottom)
+		)
+	)
 	(label "J3_D+"
-		(at 40.64 93.98 180)
+		(at 39.37 104.14 180)
 		(effects
 			(font
@@
 		)
 	)
+	(label "J3_D+"
+		(at 39.37 99.06 180)
+		(effects
+			(font
+				(size 1.27 1.27)
+			)
+			(justify right bottom)
+		)
+	)
 	(label "J3_D-"
-		(at 48.26 43.18 180)
-		(effects
-			(font
-				(size 1.27 1.27)
-			)
-			(justify right bottom)
+		(at 76.2 45.72 0)
+		(effects
+			(font
+				(size 1.27 1.27)
+			)
+			(justify left bottom)
 		)
 	)
 	(label "J3_CC1"
-		(at 66.04 93.98 0)
+		(at 67.31 93.98 0)
 		(effects
 			(font
@@
 	(global_label "U1_P2_D-"
 		(shape input)
-		(at 76.2 45.72 0)
-		(effects
-			(font
-				(size 1.27 1.27)
-			)
-			(justify left)
+		(at 46.99 43.18 180)
+		(effects
+			(font
+				(size 1.27 1.27)
+			)
+			(justify right)
 		)
 		(property "Intersheetrefs" "${INTERSHEET_REFS}"
-			(at 76.2 45.72 0)
+			(at 46.99 43.18 0)
 			(hide yes)
 			(show_name no)
@@
 	(global_label "U1_P2_D+"
 		(shape input)
-		(at 76.2 43.18 0)
-		(effects
-			(font
-				(size 1.27 1.27)
-			)
-			(justify left)
+		(at 46.99 40.64 180)
+		(effects
+			(font
+				(size 1.27 1.27)
+			)
+			(justify right)
 		)
 		(property "Intersheetrefs" "${INTERSHEET_REFS}"
-			(at 76.2 43.18 0)
+			(at 46.99 40.64 0)
 			(hide yes)
 			(show_name no)
