File: llm-kicad/04_test_validation.kicad_sch (KiCad schematic)
At the start: 28 parts

Commit message: More progress
Parts:
- removed TP9: HIL_FLT_N, TestPoint:TestPoint_Pad_D1.5mm, symbol Connector:TestPoint
- D1, D2: value SMAJ20 -> SMAJ6.5A; LCSC C115250 -> C123817
- H1, H2, H3, H4: now in the parts list
Changed lines of the file:
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@@
 	(wire
 		(pts
-			(xy 149.86 69.85) (xy 149.86 72.39)
-		)
-		(stroke
-			(width 0)
-			(type default)
-		)
-	)
-	(wire
-		(pts
 			(xy 85.09 158.75) (xy 85.09 161.29)
 		)
@@
 		)
 	)
-	(global_label "HIL_FLT_N"
-		(shape input)
-		(at 149.86 72.39 0)
-		(effects
-			(font
-				(size 1.27 1.27)
-			)
-			(justify left)
-		)
-		(property "Intersheetrefs" "${INTERSHEET_REFS}"
-			(at 149.86 72.39 0)
-			(hide yes)
-			(show_name no)
-			(do_not_autoplace no)
-			(effects
-				(font
-					(size 1.27 1.27)
-				)
-			)
-		)
-	)
 	(global_label "HIL_VBUS_EN"
 		(shape input)
@@
 		(body_style 1)
 		(exclude_from_sim no)
-		(in_bom no)
+		(in_bom yes)
 		(on_board yes)
 		(in_pos_files yes)
@@
 		(body_style 1)
 		(exclude_from_sim no)
-		(in_bom no)
+		(in_bom yes)
 		(on_board yes)
 		(in_pos_files yes)
@@
 			)
 		)
-		(property "Value" "SMAJ20"
+		(property "Value" "SMAJ6.5A"
 			(at 39.37 149.86 0)
 			(show_name no)
@@
 			)
 		)
-		(property "LCSC" "C115250"
+		(property "LCSC" "C123817"
 			(at 41.91 149.86 0)
 			(hide yes)
@@
 		(body_style 1)
 		(exclude_from_sim no)
-		(in_bom no)
+		(in_bom yes)
 		(on_board yes)
 		(in_pos_files yes)
@@
 			)
 		)
-		(property "Value" "SMAJ20"
+		(property "Value" "SMAJ6.5A"
 			(at 27.94 149.86 0)
 			(show_name no)
@@
 			)
 		)
-		(property "LCSC" "C115250"
+		(property "LCSC" "C123817"
 			(at 30.48 149.86 0)
 			(hide yes)
@@
 		(body_style 1)
 		(exclude_from_sim no)
-		(in_bom no)
+		(in_bom yes)
 		(on_board yes)
 		(in_pos_files yes)
@@
 					(unit 1)
 				)
-			)
-		)
-	)
-	(symbol
-		(lib_id "Connector:TestPoint")
-		(at 149.86 69.85 0)
-		(unit 1)
-		(body_style 1)
-		(exclude_from_sim no)
-		(in_bom yes)
-		(on_board yes)
-		(in_pos_files yes)
-		(dnp no)
-		(property "Reference" "TP9"
-			(at 149.86 62.992 0)
-			(show_name no)
-			(do_not_autoplace no)
-			(effects
-				(font
-					(size 1.27 1.27)
-				)
-			)
-		)
-		(property "Value" "HIL_FLT_N"
-			(at 149.86 64.77 0)
-			(show_name no)
-			(do_not_autoplace no)
-			(effects
-				(font
-					(size 1.27 1.27)
-				)
-			)
-		)
-		(property "Footprint" "TestPoint:TestPoint_Pad_D1.5mm"
-			(at 149.86 69.85 0)
-			(hide yes)
-			(show_name no)
-			(do_not_autoplace no)
-			(effects
-				(font
-					(size 1.27 1.27)
-				)
-			)
-		)
-		(property "Datasheet" ""
-			(at 149.86 69.85 0)
-			(hide yes)
-			(show_name no)
-			(do_not_autoplace no)
-			(effects
-				(font
-					(size 1.27 1.27)
-				)
-			)
-		)
-		(property "Description" "test point"
-			(at 149.86 69.85 0)
-			(hide yes)
-			(show_name no)
-			(do_not_autoplace no)
-			(effects
-				(font
-					(size 1.27 1.27)
-				)
-			)
-		)
-		(pin "1"
-		)
-		(instances
-			(project "llm-kicad"
-				(path "/359235dd-5d26-44dd-816b-e50cf2415bb3/70a84e5a-da0c-48ec-8ad4-4d03aebcafb4"
-					(reference "TP9")
-					(unit 1)
-				)
