File: llm-kicad/01_power_cc.kicad_sch (KiCad schematic)
At the start: 41 parts, among them J2 TYPE-C-31-M-17, Q2 BSS138P,215, Q3 BSS138P,215, U11 TPD4E05U06DQAR, U14 TPS2121RUXR, U4 TPS259470LRPWR, U8 TLV76733DRVR

Commit message: More progress
Parts:
- removed J2: TYPE-C-31-M-17, Connector_USB:USB_C_Receptacle_HRO_TYPE-C-31-M-17, symbol Connector:USB_C_Receptacle_USB2.0_16P
- added J2: TYPE-C-31-M-17, Connector_USB:USB_C_Receptacle_HRO_TYPE-C-31-M-17, symbol Connector:USB_C_Receptacle_PowerOnly_6P
- C5: value 47uF 25V -> 100uF 10V
- R28: value 100k -> 10k; LCSC C25741 -> C25744
- R32: value 15.4k 1% -> 24k; footprint Resistor_SMD:R_0603_1608Metric -> Resistor_SMD:R_0402_1005Metric; LCSC C2933150 -> C25769
- R33, R34: LCSC C11702 -> C25744
Connections:
- net GND: now also J2.A12 (GND), J2.B12 (GND), J2.SH (SHIELD)
- net J2_CC1: now also U11.10 (NC), J2.A5 (CC1)
- net J2_CC2: now also U11.9 (NC), J2.B5 (CC2)
- net VBUS_PWR: now also J2.A9 (VBUS), J2.B9 (VBUS)
- no-connect marks 14 -> 6
Other:
- moved on the sheet: R3, R4

Commit message: Update before fixing M10
Parts:
- C5: value 100uF 10V -> 47uF 10V
Changed lines of the file:
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@@
 			)
 		)
-		(property "Value" "100uF 10V"
+		(property "Value" "47uF 10V"
 			(at 70.485 139.7 0)
 			(show_name no)
