File: llm-kicad/01_power_cc.kicad_sch (KiCad schematic)
At the start: 41 parts, among them J2 TYPE-C-31-M-17, Q2 BSS138P,215, Q3 BSS138P,215, U11 TPD4E05U06DQAR, U14 TPS2121RUXR, U4 TPS259470LRPWR, U8 TLV76733DRVR

Commit message: Fixed incorrect footprint and added external GPIO
Parts:
- removed R70, R71, R73, R74: 100k 0402, Resistor_SMD:R_0402_1005Metric, symbol Device:R
- removed R72, R75: 1k 0402, Resistor_SMD:R_0402_1005Metric, symbol Device:R
- U4: footprint TPS259470ARPWR:RPW0010A-MFG -> TPS259470ARPWR:TPS259470LRPWR
Connections:
- net +3.3V: now also R33.2; no longer R33.1
- net U14_ST: now also R33.1; no longer R33.2
Other:
- note removed: "Sense If J1 and J2 has power"
- moved on the sheet: R33

Commit message: Fixed namning of some components
Remove footprint name
Parts:
- C16: value 1uF 0402 25V -> 1uF 25V
- C17: value 10uF 0805 25V -> 10uF 25V
- C18: value 100nF 0402 -> 100nF
- R3, R4: value 5.1k 0402 -> 5.1k
- R36: value 470R 0805 -> 470R
- R37: value 100k 0402 -> 100k
- R38: value 10k 0402 -> 10k
- R39: value 18k 0402 -> 18k
- R40: value 1k 0402 -> 1k
Changed lines of the file:
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@@
 			)
 		)
-		(property "Value" "5.1k 0402"
+		(property "Value" "5.1k"
 			(at 64.77 52.07 90)
 			(show_name no)
@@
 			)
 		)
-		(property "Value" "1k 0402"
+		(property "Value" "1k"
 			(at 115.57 153.67 90)
 			(show_name no)
@@
 			)
 		)
-		(property "Value" "470R 0805"
+		(property "Value" "470R"
 			(at 190.5 136.144 90)
 			(show_name no)
@@
 			)
 		)
-		(property "Value" "100k 0402"
+		(property "Value" "100k"
 			(at 180.34 135.636 90)
 			(show_name no)
@@
 			)
 		)
-		(property "Value" "10k 0402"
+		(property "Value" "10k"
 			(at 95.758 142.494 90)
 			(show_name no)
@@
 			)
 		)
-		(property "Value" "10uF 0805 25V"
+		(property "Value" "10uF 25V"
 			(at 179.832 35.052 0)
 			(show_name no)
@@
 			)
 		)
-		(property "Value" "5.1k 0402"
+		(property "Value" "5.1k"
 			(at 57.658 52.07 90)
 			(show_name no)
@@
 			)
 		)
-		(property "Value" "18k 0402"
+		(property "Value" "18k"
 			(at 95.504 159.512 90)
 			(show_name no)
@@
 			)
 		)
-		(property "Value" "100nF 0402"
+		(property "Value" "100nF"
 			(at 196.215 34.29 0)
 			(show_name no)
@@
 			)
 		)
-		(property "Value" "1uF 0402 25V"
+		(property "Value" "1uF 25V"
 			(at 129.794 34.544 0)
 			(show_name no)
