File: llm-kicad/llm-kicad.kicad_pcb (KiCad board)
At the start: 4 copper layers, 50 x 40 mm, 101 parts, among them J1 TYPE-C-31-M-12, J2 TYPE-C-31-M-17, J3 TYPE-C-31-M-12, Q2 BSS138P,215, Q3 BSS138P,215, Q6 BSS138P,215, Q7 BSS138P,215, U1 CH334F, U10 TPD4E05U06DQA, U11 TPD4E05U06DQAR, U14 TPS2121RUXR, U2 CP2102N-A02-GQFN28, U4 TPS259470LRPWR, U5 TS3USB221A, U6 SN74LVC1G125DBVR, U8 TLV76733DRVR, U9 TPD4E05U06DQA, Y1 12MHz X322512MSB4SI

Commit message: More progress
Parts:
- removed TP9: HIL_FLT_N, TestPoint:TestPoint_Pad_D1.5mm
- added C28: 100nF, Capacitor_SMD:C_0402_1005Metric, F.Cu at (169.3, 110.2)
- C23, C25: value 1uF 25V -> 4.7uF 25V; footprint Capacitor_SMD:C_0402_1005Metric -> Capacitor_SMD:C_0805_2012Metric
- C5: value 47uF 25V -> 100uF 10V
- D1, D2: value SMAJ20 -> SMAJ6.5A
- R28: value 100k -> 10k
- R32: value 15.4k 1% -> 24k; footprint Resistor_SMD:R_0603_1608Metric -> Resistor_SMD:R_0402_1005Metric
- U1: footprint Package_DFN_QFN:QFN-24-1EP_3x4mm_P0.4mm_EP1.65x2.65mm_ThermalVias -> Package_DFN_QFN:QFN-24-1EP_4x4mm_P0.5mm_EP2.6x2.6mm_ThermalVias
- Y1: value 12MHz X322512MSB4SI -> Crystal 12MHz
- moved TP5 158.9 mm to (183.2, 123.5)
- moved TP12 145.0 mm to (179.7, 96.5)
- moved TP13 143.8 mm to (181.9, 92.8)
- moved TP6 142.8 mm to (166.3, 128.3)
- moved TP7 140.5 mm to (171.6, 93.0)
- moved TP14 133.4 mm to (171.4, 99.2)
- moved R50 133.1 mm to (180.6, 128.3)
- moved LED1 131.9 mm to (179.8, 126.8)
- moved TP1 131.2 mm to (152.2, 115.9)
- moved TP4 130.1 mm to (157.7, 91.8)
- moved TP8 130.1 mm to (161.2, 87.0)
- moved TP10 129.4 mm to (161.2, 115.0)
- moved R51 129.1 mm to (176.6, 128.4), turned to 180 degrees
- moved LED2 127.7 mm to (175.8, 126.8)
- moved TP3 125.4 mm to (149.4, 96.2)
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Connections:
- U10 pad 1: /DUT Interface/J3_D+ -> /DUT Interface/J3_D-
- U10 pad 10: unconnected-(U10-NC-Pad10) -> /DUT Interface/J3_D-
- U10 pad 2: /DUT Interface/J3_D- -> /DUT Interface/J3_D+
- U10 pad 6: unconnected-(U10-NC-Pad6) -> /DUT Interface/J3_CC2
- U10 pad 7: unconnected-(U10-NC-Pad7) -> /DUT Interface/J3_CC1
- U10 pad 9: unconnected-(U10-NC-Pad9) -> /DUT Interface/J3_D+
- U11 pad 10: unconnected-(U11-NC-Pad10) -> /Power and CC/J2_CC1
- U11 pad 9: unconnected-(U11-NC-Pad9) -> /Power and CC/J2_CC2
- U2 pad 16: VBUS_UP_SNS -> VBUS_PWR_SNS
- U2 pad 17: VBUS_HIL_SNS -> HIL_CC_EN_N
- U2 pad 18: VBUS_PWR_SNS -> VBUS_HIL_SNS
- U2 pad 20: HIL_CC_EN_N -> HIL_VBUS_EN
- U2 pad 21: HIL_DATA_EN_N -> VBUS_UP_SNS
- U2 pad 22: HIL_VBUS_EN -> HIL_DATA_EN_N
- U5 pad 1: /DUT Interface/J3_D+ -> U1_P2_D+
- U5 pad 2: /DUT Interface/J3_D- -> U1_P2_D-
- U5 pad 7: U1_P2_D- -> /DUT Interface/J3_D-
- U5 pad 8: U1_P2_D+ -> /DUT Interface/J3_D+
- U9 pad 10: unconnected-(U9-NC-Pad10) -> /USB Hub and Control/J1_D-
- U9 pad 6: unconnected-(U9-NC-Pad6) -> /USB Hub and Control/J1_CC2
- U9 pad 7: unconnected-(U9-NC-Pad7) -> /USB Hub and Control/J1_CC1
- U9 pad 9: unconnected-(U9-NC-Pad9) -> /USB Hub and Control/J1_D+
- Y1 pad 2: Net-(U1-XO) -> GND
- Y1 pad 3: (no net) -> Net-(U1-XO)
- Y1 pad 4: (no net) -> GND
Routing:
- net VSYS: track 0.00 -> 62.7 mm, vias 0 -> 5
- net +3.3V: track 0.00 -> 54.0 mm, vias 0 -> 19
- net HIL_FLT_N: track 0.00 -> 50.8 mm, vias 0 -> 2
- net VBUS_HIL: track 0.00 -> 45.4 mm, vias 0 -> 11
- net VBUS_PWR: track 0.00 -> 42.6 mm, vias 0 -> 4
- net VBUS_UP: track 0.00 -> 32.7 mm
- net HIL_DATA_EN_N: track 0.00 -> 26.9 mm, vias 0 -> 2
- net VBUS_PWR_SNS: track 0.00 -> 26.2 mm, vias 0 -> 2
- net EN_HIL: track 0.00 -> 24.7 mm, vias 0 -> 2
- net HIL_CC_EN_N: track 0.00 -> 23.8 mm, vias 0 -> 2
- net /USB Hub and Control/J1_D-: track 3.47 -> 23.4 mm
- net /USB Hub and Control/J1_D+: track 3.94 -> 23.5 mm
- net HIL_VBUS_EN: track 0.00 -> 18.4 mm, vias 0 -> 4
- net GND: track 0.00 -> 16.7 mm, vias 0 -> 8
- net VBUS_HIL_SNS: track 0.00 -> 14.8 mm
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- added copper zone on B.Cu, net +3.3V
- added copper zone on F.Cu, net +3.3V
- added copper zone on In2.Cu, net +3.3V
- added copper zone on B.Cu, net GND
- added copper zone on F.Cu, net GND
- added copper zone on In1.Cu, net GND
- added copper zone on In2.Cu, net GND
- added copper zone on B.Cu, net VBUS_HIL
- added copper zone on F.Cu, net VBUS_HIL
- added copper zone on F.Cu, net VSYS

Commit message: Update before fixing M10
Parts:
- C5: value 100uF 10V -> 47uF 10V
- moved C25 5.39 mm to (170.3, 111.5)
- moved C28 0.90 mm to (169.0, 109.3), turned to 45 degrees
- moved C24 0.69 mm to (169.2, 110.5), turned to 45 degrees
- moved C23 0.50 mm to (169.7, 107.3)
Routing:
- net HIL_FLT_N: track 50.8 -> 53.3 mm
- net +3.3V: track 54.0 -> 55.9 mm
- net GND: track 16.7 -> 17.1 mm, vias 8 -> 9
