File: llm-kicad/llm-kicad.kicad_pcb (KiCad board)
At the start: 4 copper layers, 50 x 40 mm, 101 parts, among them J1 TYPE-C-31-M-12, J2 TYPE-C-31-M-17, J3 TYPE-C-31-M-12, Q2 BSS138P,215, Q3 BSS138P,215, Q6 BSS138P,215, Q7 BSS138P,215, U1 CH334F, U10 TPD4E05U06DQA, U11 TPD4E05U06DQAR, U14 TPS2121RUXR, U2 CP2102N-A02-GQFN28, U4 TPS259470LRPWR, U5 TS3USB221A, U6 SN74LVC1G125DBVR, U8 TLV76733DRVR, U9 TPD4E05U06DQA, Y1 Crystal 12MHz

Commit message: Fixed incorrect footprint and added external GPIO
Parts:
- removed R70, R71, R73, R74: 100k 0402, Resistor_SMD:R_0402_1005Metric
- removed R72, R75: 1k 0402, Resistor_SMD:R_0402_1005Metric
- removed TP13: VBUS_PWR_SNS, TestPoint:TestPoint_Pad_D1.5mm
- removed TP15: VBUS_UP_SNS, TestPoint:TestPoint_Pad_D1.5mm
- removed TP6: GND, TestPoint:TestPoint_Pad_D1.5mm
- added C2: 100pF, Capacitor_SMD:C_0402_1005Metric, F.Cu at (167.2, 123.3)
- added J4: Conn_01x02_Socket, Connector_PinHeader_2.54mm:PinHeader_1x02_P2.54mm_Vertical, F.Cu at (164.7, 127.6)
- added R76: 330R 0402, Resistor_SMD:R_0402_1005Metric, F.Cu at (154.2, 125.3)
- added R79: 10k 0402, Resistor_SMD:R_0402_1005Metric, F.Cu at (161.3, 125.2)
- added TP16: EXT_02, TestPoint:TestPoint_Pad_D1.5mm, F.Cu at (178.3, 114.8)
- added TP9: EXT_I01, TestPoint:TestPoint_Pad_D1.5mm, F.Cu at (163.8, 116.1)
- added U15: LTV-217, Package_SO:SOP-4_4.4x2.6mm_P1.27mm, F.Cu at (157.6, 127.5)
- added U3: TPD4E05U06DQA, Package_SON:USON-10_2.5x1.0mm_P0.5mm, F.Cu at (165.7, 124.8)
- TP5: footprint TestPoint:TestPoint_Pad_D1.5mm -> TestPoint:TestPoint_Pad_D2.0mm
- U1: footprint Package_DFN_QFN:QFN-24-1EP_4x4mm_P0.5mm_EP2.6x2.6mm_ThermalVias -> Package_DFN_QFN:QFN-24-1EP_4x4mm_P0.5mm_EP2.7x2.7mm
- U4: footprint TPS259470ARPWR:RPW0010A-MFG -> TPS259470ARPWR:TPS259470LRPWR
- moved TP8 14.4 mm to (174.5, 92.6)
- moved Q6 4.17 mm to (159.2, 124.0)
- moved Q7 4.17 mm to (155.1, 123.1)
- moved R45 4.17 mm to (159.3, 121.6)
- moved R46 4.17 mm to (157.1, 121.8)
- moved TP5 2.82 mm to (181.0, 121.7)
- moved R1 2.34 mm to (154.5, 119.7), turned to 0 degrees
- moved D1 1.85 mm to (149.4, 125.4), turned to 180 degrees
- moved R2 1.52 mm to (154.5, 120.7), turned to 0 degrees
- moved R44 0.80 mm to (171.0, 105.2)
- moved R43 0.79 mm to (171.7, 106.0)
- moved TP10 0.70 mm to (160.5, 115.2)
- moved C14 0.67 mm to (162.8, 93.2)
- moved R31 0.66 mm to (161.3, 92.8)
- moved C9 0.46 mm to (157.8, 96.6)
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Connections:
- R33 pad 1: +3.3V -> U14_ST
- R33 pad 2: /Power and CC/U14_ST -> +3.3V
- U14 pad 9: /Power and CC/U14_ST -> U14_ST
- U2 pad 16: VBUS_PWR_SNS -> U14_ST
- U2 pad 21: VBUS_UP_SNS -> EXT_IO0
- U2 pad 24: unconnected-(U2-~{RTS}-Pad24) -> EXT_IO1
- U2 pad 28: unconnected-(U2-~{DTR}-Pad28) -> EXT_IO2
Routing:
- net EXT_IO0: track 0.00 -> 28.2 mm, vias 0 -> 2
- net VBUS_PWR_SNS: track 26.2 -> 0.00 mm, vias 2 -> 0
- net VBUS_PWR: track 42.6 -> 24.9 mm, vias 4 -> 3
- net U14_ST: track 0.00 -> 17.3 mm, vias 0 -> 3
- net EXT_IO2: track 0.00 -> 15.7 mm, vias 0 -> 2
- net GND: track 17.1 -> 31.9 mm, vias 9 -> 17
- net +3.3V: track 55.9 -> 70.2 mm, vias 19 -> 23
- net EXT_OUT0: track 0.00 -> 13.5 mm
- net U4_ILM: track 1.35 -> 14.4 mm
- net VBUS_UP_SNS: track 8.77 -> 0.00 mm
- net HIL_FLT_N: track 53.3 -> 46.3 mm
- net EXT_IO1: track 0.00 -> 6.82 mm
- net EN_HIL: track 24.7 -> 31.4 mm
- net VBUS_HIL: track 45.4 -> 41.6 mm
- net /Power and CC/VBUS_PWR_DIV: track 2.54 -> 0.00 mm
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- added copper zone on In1.Cu, net +3.3V
Other:
- board text added: "DATA"
- board text added: "Power"
- board text added: "To DUT"
- board text added: "V2.0"
- board text added: "VBUS-HIL"

Commit message: Ready for first production
Parts:
- moved R47 3.47 mm to (166.6, 104.9)
- moved R43 1.87 mm to (171.0, 104.3)
- moved R44 1.87 mm to (170.3, 103.5)
- moved R4 0.94 mm to (150.2, 99.0)
- moved R3 0.88 mm to (150.2, 100.2)
- moved C23 0.62 mm to (169.4, 106.8), turned to 45 degrees
Routing:
- net VBUS_HIL: track 41.6 -> 21.9 mm, vias 11 -> 18
- net /USB Hub and Control/J1_D-: track 23.4 -> 27.4 mm
- net /DUT Interface/J3_D-: track 6.63 -> 10.5 mm
- net /DUT Interface/J3_D+: track 6.63 -> 10.2 mm, vias 0 -> 2
- net /USB Hub and Control/J1_D+: track 23.5 -> 26.9 mm, vias 0 -> 2
- net U4_ILM: track 14.4 -> 17.6 mm, vias 0 -> 2
- net GND: track 31.9 -> 33.4 mm, vias 17 -> 83
- net /Power and CC/J2_CC1: track 6.28 -> 7.74 mm
- net /Power and CC/J2_CC2: track 8.68 -> 10.1 mm
- net /USB Hub and Control/U2_RST_N: track 4.53 -> 3.36 mm
- net /USB Hub and Control/U2_VBUS_DIV: track 5.60 -> 6.55 mm
- net +3.3V: track 70.2 -> 69.5 mm
- net U1_P2_D-: track 12.5 -> 13.1 mm
- net VBUS_PWR: track 24.9 -> 24.6 mm, vias 3 -> 10
- net VBUS_UP: vias 0 -> 9
- added copper zone on B.Cu, net VBUS_PWR
- added copper zone on F.Cu, net VBUS_PWR
- added copper zone on B.Cu, net VBUS_UP
- added copper zone on F.Cu, net VBUS_UP
